File: ST-LINK-V2_1.kicad_pcb (KiCad board)
At the start: 2 copper layers, 50 x 20 mm, 44 parts, among them IC1 AP7333-33SAG-7, J1 USB_C_Receptacle_USB2.0_16P, J2 OUTPUT, J3 frm, Q1 MMBT3904, U1 STM32F103CBTx, Y1 8mHz

Commit message: Ver-1.1
Parts:
- removed REF** (x4): MountingHole_2.1mm, MountingHole:MountingHole_2.1mm
- moved G*** 0.30 mm to (125.7, 77.5)
Routing:
- net /T_RXD: track 26.1 -> 35.6 mm
- net /T_TXD: track 25.2 -> 32.4 mm
- net /T_SWO: track 33.3 -> 35.4 mm
- net /T_NRST: track 28.5 -> 29.7 mm
Other:
- outline, holes or cut-outs redrawn
